File: wifi_temp_sensor.kicad_pcb (KiCad board)
At the start: 2 copper layers, 50.2 x 33 mm, 9 parts, among them J1 USB_B_Mini, J2 Conn_02x04_Odd_Even, J3 Conn_01x04, J4 Conn_01x06, J6 Conn_01x01, J8 Conn_01x01, SW1 SW_DIP_x01

Commit message: semi complete schematic
Parts:
- removed 3_3VOUT1, 5VIN1, J6, J8: Conn_01x01, Connector_PinSocket_2.54mm:PinSocket_1x01_P2.54mm_Vertical
- removed J3: Conn_01x04, Connector_PinSocket_2.54mm:PinSocket_1x04_P2.54mm_Horizontal
- removed J4: Conn_01x06, Connector_PinHeader_2.54mm:PinHeader_1x06_P2.54mm_Vertical
- removed SW1: SW_DIP_x01, Button_Switch_THT:SW_PUSH_6mm
- added IC1: ESP32-C3-WROOM-02-N4, KiCad:ESP32C3WROOM02N4, F.Cu at (134.4, 67.2)
- J1: value USB_B_Mini -> USB_C_Receptacle_USB2.0; footprint Connector_USB:USB_Micro-B_Molex-105017-0001 -> Connector_USB:USB_C_Receptacle_Molex_105450-0101
- J2: value Conn_02x04_Odd_Even -> Batt_Conn; footprint Connector_PinSocket_2.54mm:PinSocket_2x04_P2.54mm_Vertical -> Connector_JST:JST_ACH_BM02B-ACHSS-GAN-ETF_1x02-1MP_P1.20mm_Vertical; moved to B.Cu
- moved J1 108.9 mm to (137.9, 112.4), turned to 0 degrees
- moved J2 77.3 mm to (127.7, 109.9), turned to 90 degrees
Connections:
- J2 pad 2: ESP_Tx -> V_BAT
Routing:
- net GND: track 98.0 -> 0.00 mm
- net +3.3V: track 50.7 -> 0.00 mm
- net +5V: track 35.8 -> 0.00 mm
- net SCL: track 33.1 -> 0.00 mm
- net ESP_Rx: track 29.7 -> 0.00 mm
- net ESP_Tx: track 26.7 -> 0.00 mm
- net SDA: track 23.2 -> 0.00 mm
- net unconnected-(J1-Shield-Pad6): track 12.1 -> 0.00 mm
Other:
- board outline removed

Commit message: fixes, still in progress
Parts:
- removed IC1: ESP32-C3-WROOM-02-N4, KiCad:ESP32C3WROOM02N4
- removed J1: USB_C_Receptacle_USB2.0, Connector_USB:USB_C_Receptacle_Molex_105450-0101
- added B_CHARGER1: BQ21040DBVR, TI BQ21040:SOT95P280X145-6N, F.Cu at (95.4, 65.0)
- added B_SWITCH1: SW_SPST, Button_Switch_SMD:SW_SPDT_CK-JS102011SAQN, F.Cu at (116.6, 114.3)
- added C1: C_Small, Capacitor_SMD:C_0402_1005Metric, F.Cu at (116.8, 90.5)
- added C2: C_Small, Capacitor_SMD:C_0402_1005Metric, F.Cu at (116.8, 92.5)
- added C3: C_Small, Capacitor_SMD:C_0402_1005Metric, F.Cu at (116.8, 94.4)
- added D1: D_Schottky, Diode_SMD:D_0805_2012Metric, F.Cu at (107.5, 99.0)
- added D2: LED_Small, LED_SMD:LED_0402_1005Metric, F.Cu at (117.1, 96.4)
- added L1: L_Small, Inductor_SMD:L_0805_2012Metric, F.Cu at (112.8, 99.8)
- added MCU1: ESP32-C3-WROOM-02-N4, Nordic ESP32-C3-WROOM-02-N4:ESP32C3WROOM02N4, F.Cu at (162.7, 90.2)
- added PSU1: TLV62569DBV, Package_TO_SOT_SMD:SOT-23-5, F.Cu at (95.4, 69.5)
- added Q1: DMG3414U, Package_TO_SOT_SMD:SOT-23, F.Cu at (112.9, 91.7)
- added Q2: DMG3414U, Package_TO_SOT_SMD:SOT-23, F.Cu at (112.9, 96.2)
- added R1: R_Small, Resistor_SMD:R_0402_1005Metric, F.Cu at (112.0, 80.5)
- added R10: R_Small, Resistor_SMD:R_0402_1005Metric, F.Cu at (114.9, 88.5)
- added R2: R_Small, Resistor_SMD:R_0402_1005Metric, F.Cu at (112.0, 82.5)
- added R3: 10k, Resistor_SMD:R_0402_1005Metric, F.Cu at (130.9, 66.0)
- added R4: 10k, Resistor_SMD:R_0402_1005Metric, F.Cu at (130.9, 64.8)
- added R5: R_Small, Resistor_SMD:R_0402_1005Metric, F.Cu at (112.0, 88.5)
- added R6: R_Small, Resistor_SMD:R_0402_1005Metric, F.Cu at (114.9, 80.5)
- added R7: R_Small, Resistor_SMD:R_0402_1005Metric, F.Cu at (114.9, 82.5)
- added R8: R_Small, Resistor_SMD:R_0402_1005Metric, F.Cu at (114.9, 84.5)
- added R9: R_Small, Resistor_SMD:R_0402_1005Metric, F.Cu at (114.9, 86.5)
- added T_H_SENSOR1: SHT4x, Sensor_Humidity:Sensirion_DFN-4_1.5x1.5mm_P0.8mm_SHT4x_NoCentralPad, F.Cu at (136.5, 65.0)
- added USB_CONN1: USB_C_Receptacle_USB2.0, Connector_USB:USB_C_Receptacle_Molex_105450-0101, F.Cu at (139.7, 112.4)
Connections:
- J2 pad 2: V_BAT -> Net-(B_SWITCH1-A)
Routing:
- net SDC: track 0.00 -> 4.58 mm
- net SDA: track 0.00 -> 4.38 mm
