File: wifi_temp_sensor.kicad_sch (KiCad schematic)
At the start: 25 parts, among them IC1 ESP32-C3-WROOM-02-N4, IC2 BQ21040DBVR, J1 USB_C_Receptacle_USB2.0, J2 Batt_Conn, Q1 BF545A, Q2 BF545A, SW1 SW_SPST, U1 SHT4x, U2 TLV62569DBV

Commit message: fixes, still in progress
Parts:
- removed Q1, Q2: BF545A, Package_TO_SOT_SMD:SOT-23, symbol Transistor_FET:BF545A
- added C4, C5: C_Small, symbol Device:C_Small
- added F1: Polyfuse_Small, symbol Device:Polyfuse_Small
- added J1: TC2030-IDC-NL, TC2030-IDC-NL:TAG_TC2030-IDC-NL, symbol TC2030-IDC-NL:TC2030-IDC-NL
- added Q1: DMG3414U, Package_TO_SOT_SMD:SOT-23, symbol Transistor_FET:DMG3414U
- B_SWITCH1: renamed from SW1; footprint (none) -> Button_Switch_SMD:SW_SPDT_CK-JS102011SAQN
- C1, C2, C3: footprint (none) -> Capacitor_SMD:C_0402_1005Metric
- D1: footprint (none) -> Diode_SMD:D_0805_2012Metric
- D2: footprint (none) -> LED_SMD:LED_0402_1005Metric
- L1: footprint (none) -> Inductor_SMD:L_0805_2012Metric
- R1, R10, R2, R3, R4, R5, R6, R7, R8, R9: footprint (none) -> Resistor_SMD:R_0402_1005Metric
- renumbered IC2 to B_CHARGER1, IC1 to MCU1, U2 to PSU1, U1 to T_H_SENSOR1, J1 to USB_CONN1
Connections:
- net D+: now also C5.1
- net D-: now also C4.1
- net GND: now also R1.2, C4.2, C5.2
- net VBAT_MEAS_EN: now also Q1.1 (G)
- net V_BAT: now also Q1.3 (D); no longer R10.1, R2.1
- net V_USB: now also R10.1, F1.1; no longer USB_CONN1.A4 (VBUS), USB_CONN1.A9 (VBUS), USB_CONN1.B4 (VBUS), USB_CONN1.B9 (VBUS)
- new net: F1.2, USB_CONN1.A4 (VBUS), USB_CONN1.A9 (VBUS), USB_CONN1.B4 (VBUS), USB_CONN1.B9 (VBUS)
- new net: Q1.2 (S), R2.1
Other:
- note added: "I have no idea how to pick the inductor component"
- note added: "This might be the wrong type of MOSFET"
- moved on the sheet: B_CHARGER1, B_SWITCH1, C1, C2, C3, D1, D2, J2, L1, PSU1, R1, R10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

Commit message: mods
Connections:
- net +3.3V: now also MCU1.2 (EN)
Changed lines of the file:
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@@
   (junction (at 261.62 86.36) (diameter 0) (color 0 0 0 0)
+  )
+  (junction (at 38.1 154.94) (diameter 0) (color 0 0 0 0)
   )
   (junction (at 48.26 101.6) (diameter 0) (color 0 0 0 0)
@@
     (stroke (width 0) (type default))
   )
-  (wire (pts (xy 41.91 154.94) (xy 25.4 154.94))
+  (wire (pts (xy 41.91 154.94) (xy 38.1 154.94))
     (stroke (width 0) (type default))
   )
@@
     (stroke (width 0) (type default))
   )
+  (wire (pts (xy 38.1 157.48) (xy 38.1 154.94))
+    (stroke (width 0) (type default))
+  )
   (wire (pts (xy 78.74 177.8) (xy 78.74 180.34))
     (stroke (width 0) (type default))
@@
     (stroke (width 0) (type default))
   )
+  (wire (pts (xy 38.1 154.94) (xy 25.4 154.94))
+    (stroke (width 0) (type default))
+  )
   (wire (pts (xy 229.87 135.89) (xy 234.95 135.89))
     (stroke (width 0) (type default))
@@
     (stroke (width 0) (type default))
   )
+  (wire (pts (xy 41.91 157.48) (xy 38.1 157.48))
+    (stroke (width 0) (type default))
+  )
