File: wifi_temp_sensor.kicad_sch (KiCad schematic)
At the start: 47 parts, among them IC2 BQ21040DBVR, J2 Batt_Conn, J3 Conn_02x03_Odd_Even, P1 USB_C_Plug_USB2.0, Q1 SSM6L09FUTE85LF, Q2 AO3401A, Q3 BSS214NW, SW1 SW_SPST, U1 ESP32-C3-WROOM-02, U2 SHT4x, U3 WE-TVS-82400102, U4 LD1117S33TR_SOT223

Commit message: Notes and initial PCB layout
Parts:
- C1, C12, C4, C5, C7, C8: footprint (none) -> Capacitor_SMD:C_0603_1608Metric
- D1: footprint (none) -> Diode_SMD:D_0603_1608Metric
- F1: footprint (none) -> Fuse:Fuse_0603_1608Metric
- R1, R10, R12, R13, R15, R16, R17, R19, R2, R20, R3, R4, R9: footprint (none) -> Resistor_SMD:R_0603_1608Metric
- SW1: footprint (none) -> Button_Switch_SMD:SW_SPDT_CK-JS102011SAQN
Connections:
- no-connect marks 0 -> 1
Other:
- note added: "Has to be a P-Channel. It will turn OFF when the V_USB is present"
- note added: "I'm missing something basic. Is the 100nF cap for decoupling?"
- note added: "Is this for diag / reporting?"
- note added: "Not sure what pin 16 is for?"
- note added: "Not sure where this is supposed to connect"
- note added: "Why use a p-channel n-channel package here?"
Changed lines of the file:
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@@
   (junction (at 252.73 87.63) (diameter 0) (color 0 0 0 0)
   )
+  (no_connect (at 271.78 62.23))
   (wire (pts (xy 207.01 24.13) (xy 209.55 24.13))
     (stroke (width 0) (type default))
@@
     (fill (type none))
     (effects (font (size 1.27 1.27)) (justify left top))
+  )
+  (text "Is this for diag / reporting?" (at 105.41 72.39 0)
+    (effects (font (size 1.27 1.27)) (justify left bottom))
+  )
+  (text "Why use a p-channel n-channel package here?" (at 69.85 19.05 0)
+    (effects (font (size 1.27 1.27)) (justify left bottom))
+  )
+  (text "Not sure what pin 16 is for?" (at 140.97 158.75 0)
+    (effects (font (size 1.27 1.27)) (justify left bottom))
+  )
+  (text "Not sure where this is supposed to connect" (at 48.26 90.17 0)
+    (effects (font (size 1.27 1.27)) (justify left bottom))
+  )
+  (text "I'm missing something basic.\nIs the 100nF cap for decoupling?"
+    (at 102.87 96.52 0)
+    (effects (font (size 1.27 1.27)) (justify left bottom))
+  )
+  (text "I'm missing something basic.\nIs the 100nF cap for decoupling?"
+    (at 160.02 53.34 0)
+    (effects (font (size 1.27 1.27)) (justify left bottom))
+  )
+  (text "Has to be a P-Channel. It will turn OFF when the V_USB is present"
+    (at 186.69 69.85 0)
+    (effects (font (size 1.27 1.27)) (justify left bottom))
   )
   (text "Alt: USBLC6-2SC6\n" (at 243.84 50.8 0)
@@
       (effects (font (size 1.27 1.27)) (justify left))
     )
-    (property "Footprint" "" (at 97.79 81.28 0)
+    (property "Footprint" "Resistor_SMD:R_0603_1608Metric" (at 97.79 81.28 0)
       (effects (font (size 1.27 1.27)) hide)
     )
@@
       (effects (font (size 1.27 1.27)) (justify left))
     )
-    (property "Footprint" "" (at 228.6 93.98 0)
+    (property "Footprint" "Capacitor_SMD:C_0603_1608Metric" (at 228.6 93.98 0)
       (effects (font (size 1.27 1.27)) hide)
     )
@@
       (effects (font (size 1.27 1.27)))
     )
-    (property "Footprint" "" (at 232.41 25.4 0)
+    (property "Footprint" "Fuse:Fuse_0603_1608Metric" (at 232.41 25.4 0)
       (effects (font (size 1.27 1.27)) (justify left) hide)
     )
@@
       (effects (font (size 1.27 1.27)))
     )
-    (property "Footprint" "" (at 218.44 78.74 0)
+    (property "Footprint" "Diode_SMD:D_0603_1608Metric" (at 218.44 78.74 0)
       (effects (font (size 1.27 1.27)) hide)
     )
@@
       (effects (font (size 1.27 1.27)) (justify left))
     )
-    (property "Footprint" "" (at 179.07 133.35 0)
+    (property "Footprint" "Resistor_SMD:R_0603_1608Metric" (at 179.07 133.35 0)
       (effects (font (size 1.27 1.27)) hide)
     )
@@
       (effects (font (size 1.27 1.27)) (justify left))
     )
-    (property "Footprint" "" (at 97.79 68.58 0)
+    (property "Footprint" "Resistor_SMD:R_0603_1608Metric" (at 97.79 68.58 0)
       (effects (font (size 1.27 1.27)) hide)
     )
@@
       (effects (font (size 1.27 1.27)))
     )
-    (property "Footprint" "" (at 237.49 31.75 0)
+    (property "Footprint" "Resistor_SMD:R_0603_1608Metric" (at 237.49 31.75 0)
       (effects (font (size 1.27 1.27)) hide)
     )
@@
       (effects (font (size 1.27 1.27)) (justify left))
     )
-    (property "Footprint" "" (at 105.41 138.43 0)
+    (property "Footprint" "Resistor_SMD:R_0603_1608Metric" (at 105.41 138.43 0)
       (effects (font (size 1.27 1.27)) hide)
     )
@@
       (effects (font (size 1.27 1.27)) (justify left))
     )
-    (property "Footprint" "" (at 207.01 48.26 0)
+    (property "Footprint" "Capacitor_SMD:C_0603_1608Metric" (at 207.01 48.26 0)
       (effects (font (size 1.27 1.27)) hide)
     )
@@
       (effects (font (size 1.27 1.27)) (justify left))
     )
-    (property "Footprint" "" (at 78.74 72.39 0)
+    (property "Footprint" "Resistor_SMD:R_0603_1608Metric" (at 78.74 72.39 0)
       (effects (font (size 1.27 1.27)) hide)
     )
@@
       (effects (font (size 1.27 1.27)) (justify left))
     )
-    (property "Footprint" "" (at 205.74 140.97 0)
+    (property "Footprint" "Capacitor_SMD:C_0603_1608Metric" (at 205.74 140.97 0)
       (effects (font (size 1.27 1.27)) hide)
     )
@@
       (effects (font (size 1.27 1.27)) (justify left))
     )
-    (property "Footprint" "" (at 113.03 138.43 0)
+    (property "Footprint" "Resistor_SMD:R_0603_1608Metric" (at 113.03 138.43 0)
       (effects (font (size 1.27 1.27)) hide)
     )
@@
       (effects (font (size 1.27 1.27)) (justify left))
     )
-    (property "Footprint" "" (at 182.88 133.35 0)
+    (property "Footprint" "Resistor_SMD:R_0603_1608Metric" (at 182.88 133.35 0)
       (effects (font (size 1.27 1.27)) hide)
     )
@@
       (effects (font (size 1.27 1.27)) (justify left))
     )
-    (property "Footprint" "" (at 144.78 35.56 0)
+    (property "Footprint" "Resistor_SMD:R_0603_1608Metric" (at 144.78 35.56 0)
       (effects (font (size 1.27 1.27)) hide)
     )
@@
       (effects (font (size 1.27 1.27)) (justify left))
     )
-    (property "Footprint" "" (at 45.72 88.9 0)
+    (property "Footprint" "Resistor_SMD:R_0603_1608Metric" (at 45.72 88.9 0)
       (effects (font (size 1.27 1.27)) hide)
     )
@@
       (effects (font (size 1.27 1.27)) (justify left))
     )
-    (property "Footprint" "" (at 215.9 48.26 0)
+    (property "Footprint" "Capacitor_SMD:C_0603_1608Metric" (at 215.9 48.26 0)
       (effects (font (size 1.27 1.27)) hide)
     )
@@
       (effects (font (size 1.27 1.27)) (justify left))
     )
-    (property "Footprint" "" (at 110.49 81.28 0)
+    (property "Footprint" "Capacitor_SMD:C_0603_1608Metric" (at 110.49 81.28 0)
       (effects (font (size 1.27 1.27)) hide)
     )
@@
       (effects (font (size 1.27 1.27)))
     )
-    (property "Footprint" "" (at 237.49 29.21 0)
+    (property "Footprint" "Resistor_SMD:R_0603_1608Metric" (at 237.49 29.21 0)
       (effects (font (size 1.27 1.27)) hide)
     )
@@
       (effects (font (size 1.27 1.27)) (justify left))
     )
-    (property "Footprint" "" (at 157.48 45.72 0)
+    (property "Footprint" "Capacitor_SMD:C_0603_1608Metric" (at 157.48 45.72 0)
       (effects (font (size 1.27 1.27)) hide)
     )
@@
       (effects (font (size 1.27 1.27)) (justify left))
     )
-    (property "Footprint" "" (at 144.78 45.72 0)
+    (property "Footprint" "Resistor_SMD:R_0603_1608Metric" (at 144.78 45.72 0)
       (effects (font (size 1.27 1.27)) hide)
     )
@@
       (effects (font (size 1.27 1.27)) (justify left))
     )
-    (property "Footprint" "" (at 120.65 138.43 0)
+    (property "Footprint" "Resistor_SMD:R_0603_1608Metric" (at 120.65 138.43 0)
       (effects (font (size 1.27 1.27)) hide)
     )
@@
       (effects (font (size 1.27 1.27)))
     )
-    (property "Footprint" "" (at 40.64 27.94 0)
-      (effects (font (size 1.27 1.27)) hide)
-    )
+    (property "Footprint" "Button_Switch_SMD:SW_SPDT_CK-JS102011SAQN" (at 40.64 27.94 0)
+      (effects (font (size 1.27 1.27)) hide)
+    )
