File: hardware/wifi_temp_sensor.kicad_sch (KiCad schematic)
At the start: 46 parts, among them IC2 BQ21040DBVR, J2 Batt_Conn, J3 Conn_02x03_Odd_Even, P1 USB_C_Plug_USB2.0, Q1 SSM6L09FUTE85LF, Q2 AO3401A, Q3 BSS214NW, SW1 SW_SPST, SW2 SW_Push, U1 ESP32-C3-WROOM-02, U2 SHT4x, U3 WE-TVS-82400102, U4 LD1117S33TR_SOT223

Commit message: Fixed up errors, ready for review
Parts:
- added R7: 10k, Resistor_SMD:R_0603_1608Metric, symbol Device:R_Small
Connections:
- net VBAT_MEAS_EN: now also R16.2, U1.7 (GPIO8); no longer U1.4 (GPIO5/ADC2_CH0)
- net V_USB: now also R7.1
- net at IC2.1 (TS), Q3.3 (D): now also R7.2
- removed net CHG_ENABLE: Q3.1 (G), R16.2, U1.7 (GPIO8)
- new net ~{CHG_ENABLE}: Q3.1 (G), U1.4 (GPIO5/ADC2_CH0)
Changed lines of the file:
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@@
   (junction (at 73.66 27.94) (diameter 0) (color 0 0 0 0)
   )
+  (junction (at 120.65 176.53) (diameter 0) (color 0 0 0 0)
+  )
   (junction (at 215.9 36.83) (diameter 0) (color 0 0 0 0)
   )
@@
   (junction (at 218.44 24.13) (diameter 0) (color 0 0 0 0)
   )
+  (junction (at 36.83 63.5) (diameter 0) (color 0 0 0 0)
+  )
   (junction (at 207.01 41.91) (diameter 0) (color 0 0 0 0)
   )
@@
   )
   (junction (at 228.6 87.63) (diameter 0) (color 0 0 0 0)
-  )
-  (junction (at 120.65 176.53) (diameter 0) (color 0 0 0 0)
   )
   (junction (at 97.79 76.2) (diameter 0) (color 0 0 0 0)
@@
     (stroke (width 0) (type default))
   )
+  (wire (pts (xy 36.83 53.34) (xy 36.83 55.88))
+    (stroke (width 0) (type default))
+  )
   (wire (pts (xy 139.7 91.44) (xy 139.7 97.79))
     (stroke (width 0) (type default))
@@
     (stroke (width 0) (type default))
   )
+  (wire (pts (xy 120.65 176.53) (xy 125.73 176.53))
+    (stroke (width 0) (type default))
+  )
   (wire (pts (xy 219.71 87.63) (xy 227.33 87.63))
     (stroke (width 0) (type default))
@@
     (stroke (width 0) (type default))
   )
-  (wire (pts (xy 120.65 176.53) (xy 125.73 176.53))
-    (stroke (width 0) (type default))
-  )
   (wire (pts (xy 241.3 41.91) (xy 248.92 41.91))
     (stroke (width 0) (type default))
@@
     (stroke (width 0) (type default))
   )
+  (wire (pts (xy 101.6 168.91) (xy 125.73 168.91))
+    (stroke (width 0) (type default))
+  )
   (wire (pts (xy 214.63 104.14) (xy 214.63 106.68))
     (stroke (width 0) (type default))
@@
     (stroke (width 0) (type default))
   )
+  (wire (pts (xy 36.83 60.96) (xy 36.83 63.5))
+    (stroke (width 0) (type default))
+  )
   (wire (pts (xy 261.62 85.09) (xy 261.62 87.63))
     (stroke (width 0) (type default))
@@
     (stroke (width 0) (type default))
   )
+  (wire (pts (xy 43.18 53.34) (xy 36.83 53.34))
+    (stroke (width 0) (type default))
+  )
   (wire (pts (xy 87.63 71.12) (xy 87.63 76.2))
     (stroke (width 0) (type default))
@@
   )
   (wire (pts (xy 234.95 143.51) (xy 247.65 143.51))
-    (stroke (width 0) (type default))
-  )
-  (wire (pts (xy 101.6 168.91) (xy 125.73 168.91))
     (stroke (width 0) (type default))
   )
@@
     )
   )
-  (global_label "CHG_ENABLE" (shape input) (at 49.53 86.36 0) (fields_autoplaced)
+  (global_label "~{CHG_ENABLE}" (shape input) (at 49.53 86.36 0) (fields_autoplaced)
     (effects (font (size 1.27 1.27)) (justify left))
-    (property "Intersheetrefs" "${INTERSHEET_REFS}" (at 64.2891 86.36 0)
+    (property "Intersheetrefs" "${INTERSHEET_REFS}" (at 64.3685 86.36 0)
       (effects (font (size 1.27 1.27)) (justify left) hide)
     )
@@
     )
   )
+  (global_label "V_USB" (shape input) (at 43.18 53.34 0) (fields_autoplaced)
+    (effects (font (size 1.27 1.27)) (justify left))
+    (property "Intersheetrefs" "${INTERSHEET_REFS}" (at 52.0314 53.34 0)
+      (effects (font (size 1.27 1.27)) (justify left) hide)
+    )
+  )
   (global_label "EN" (shape bidirectional) (at 234.95 140.97 180) (fields_autoplaced)
     (effects (font (size 1.27 1.27)) (justify right))
@@
     )
   )
-  (global_label "VBAT_MEAS_EN" (shape output) (at 125.73 168.91 0) (fields_autoplaced)
+  (global_label "VBAT_MEAS_EN" (shape output) (at 125.73 176.53 0) (fields_autoplaced)
     (effects (font (size 1.27 1.27)) (justify left))
-    (property "Intersheetrefs" "${INTERSHEET_REFS}" (at 142.3638 168.91 0)
+    (property "Intersheetrefs" "${INTERSHEET_REFS}" (at 142.3638 176.53 0)
       (effects (font (size 1.27 1.27)) (justify left) hide)
     )
@@
     )
   )
-  (global_label "CHG_ENABLE" (shape output) (at 125.73 176.53 0) (fields_autoplaced)
+  (global_label "~{CHG_ENABLE}" (shape output) (at 125.73 168.91 0) (fields_autoplaced)
     (effects (font (size 1.27 1.27)) (justify left))
-    (property "Intersheetrefs" "${INTERSHEET_REFS}" (at 140.4891 176.53 0)
+    (property "Intersheetrefs" "${INTERSHEET_REFS}" (at 140.5685 168.91 0)
       (effects (font (size 1.27 1.27)) (justify left) hide)
     )
@@
         )
       )
+    )
+  )
+  (symbol (lib_id "Device:R_Small") (at 36.83 58.42 0) (unit 1)
+    (in_bom yes) (on_board yes) (dnp no) (fields_autoplaced)
+    (property "Reference" "R7" (at 39.37 57.785 0)
+      (effects (font (size 1.27 1.27)) (justify left))
+    )
+    (property "Value" "10k" (at 39.37 60.325 0)
+      (effects (font (size 1.27 1.27)) (justify left))
+    )
+    (property "Footprint" "Resistor_SMD:R_0603_1608Metric" (at 36.83 58.42 0)
+      (effects (font (size 1.27 1.27)) hide)
+    )
+    (property "Datasheet" "~" (at 36.83 58.42 0)
+      (effects (font (size 1.27 1.27)) hide)
+    )
+    (pin "1")
+    (pin "2")
+    (instances
+      (project "wifi_temp_sensor"
+        (path "/f6c77997-b71a-421e-9dbe-7ca9e2d5ccfe"
+          (reference "R7") (unit 1)
+        )
+      )
