File: hardware/wifi_temp_sensor.kicad_pcb (KiCad board)
At the start: 2 copper layers, 50.8 x 45.7 mm, 12 parts, among them J1 USB_B_Mini, J2 ESP8266, J3 TempSensor, J4 Prog, J5 Aux_I2C, SW1 BootMode, U2 AZ1117-3.3

Commit message: small re-route
Parts:
- moved SW1 7.91 mm to (231.2, 37.2), turned to 180 degrees
Routing:
- net ESP_Rx: track 21.2 -> 16.9 mm
- net SCL: track 60.3 -> 58.5 mm
- net +3.3V: track 54.1 -> 55.6 mm, vias 0 -> 2
Changed lines of the file:
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@@
   )
   (footprint "Button_Switch_THT:SW_PUSH_6mm" (layer "F.Cu")
-    (at 224.715 32.675)
+    (at 231.215 37.175 180)
     (descr "https://www.omron.com/ecb/products/pdf/en-b3f.pdf")
     (tags "tact sw push 6mm")
@@
         (effects (font (size 1 1) (thickness 0.15)))
     )
-    (fp_text value "BootMode" (at 3.75 6.695) (layer "F.SilkS")
+    (fp_text value "BootMode" (at 4.52 6.695) (layer "F.SilkS")
         (effects (font (size 1 1) (thickness 0.15)))
     )
@@
     (fp_circle (center 3.25 2.25) (end 1.25 2.5)
       (stroke (width 0.1) (type solid)) (fill none) (layer "F.Fab"))
-    (pad "1" thru_hole circle (at 0 0 90) (size 2 2) (drill 1.1) (layers "*.Cu" "*.Mask")
+    (pad "1" thru_hole circle (at 0 0 270) (size 2 2) (drill 1.1) (layers "*.Cu" "*.Mask")
       (net 10 "SCL") (pintype "passive"))
-    (pad "1" thru_hole circle (at 6.5 0 90) (size 2 2) (drill 1.1) (layers "*.Cu" "*.Mask")
+    (pad "1" thru_hole circle (at 6.5 0 270) (size 2 2) (drill 1.1) (layers "*.Cu" "*.Mask")
       (net 10 "SCL") (pintype "passive"))
-    (pad "2" thru_hole circle (at 0 4.5 90) (size 2 2) (drill 1.1) (layers "*.Cu" "*.Mask")
+    (pad "2" thru_hole circle (at 0 4.5 270) (size 2 2) (drill 1.1) (layers "*.Cu" "*.Mask")
       (net 6 "GND") (pintype "passive"))
-    (pad "2" thru_hole circle (at 6.5 4.5 90) (size 2 2) (drill 1.1) (layers "*.Cu" "*.Mask")
+    (pad "2" thru_hole circle (at 6.5 4.5 270) (size 2 2) (drill 1.1) (layers "*.Cu" "*.Mask")
       (net 6 "GND") (pintype "passive"))
     (model "${KICAD6_3DMODEL_DIR}/Button_Switch_THT.3dshapes/SW_PUSH_6mm.wrl"
@@
     (stroke (width 0.1) (type default)) (layer "Edge.Cuts"))
   (segment (start 201.93 43.18) (end 201.93 46.15) (width 1) (layer "F.Cu") (net 1))
+  (segment (start 210.195 63.5) (end 210.185 63.49) (width 0.5) (layer "F.Cu") (net 1))
   (segment (start 216.535 56.085) (end 216.535 46.67) (width 1) (layer "F.Cu") (net 1))
+  (segment (start 213.995 60.325) (end 213.995 58.625) (width 0.5) (layer "F.Cu") (net 1))
   (segment (start 210.185 58.41) (end 213.78 58.41) (width 1) (layer "F.Cu") (net 1))
   (segment (start 213.995 58.625) (end 216.535 56.085) (width 1) (layer "F.Cu") (net 1))
@@
   (segment (start 208.28 43.18) (end 208.28 46.15) (width 1) (layer "F.Cu") (net 1))
   (segment (start 213.78 58.41) (end 213.995 58.625) (width 1) (layer "F.Cu") (net 1))
-  (segment (start 213.995 59.68) (end 213.995 58.625) (width 1) (layer "F.Cu") (net 1))
   (segment (start 220.345 45.72) (end 218.3975 45.72) (width 0.5) (layer "F.Cu") (net 1))
+  (segment (start 212.715 63.49) (end 212.725 63.5) (width 0.25) (layer "F.Cu") (net 1))
   (segment (start 215.9 45.72) (end 218.3975 45.72) (width 0.5) (layer "F.Cu") (net 1))
   (segment (start 208.71 45.72) (end 218.3975 45.72) (width 1) (layer "F.Cu") (net 1))
+  (segment (start 212.725 63.5) (end 210.195 63.5) (width 0.5) (layer "F.Cu") (net 1))
   (segment (start 221.66 46.125) (end 220.75 46.125) (width 0.5) (layer "F.Cu") (net 1))
-  (segment (start 210.185 63.49) (end 213.995 59.68) (width 1) (layer "F.Cu") (net 1))
   (segment (start 208.28 46.15) (end 208.71 45.72) (width 1) (layer "F.Cu") (net 1))
   (segment (start 220.75 46.125) (end 220.345 45.72) (width 0.5) (layer "F.Cu") (net 1))
+  (via (at 213.995 60.325) (size 0.8) (drill 0.4) (layers "F.Cu" "B.Cu") (free) (net 1))
+  (via (at 212.725 63.5) (size 0.8) (drill 0.4) (layers "F.Cu" "B.Cu") (free) (net 1))
+  (segment (start 212.725 63.5) (end 212.725 61.595) (width 0.5) (layer "B.Cu") (net 1))
+  (segment (start 212.725 61.595) (end 213.995 60.325) (width 0.5) (layer "B.Cu") (net 1))
   (segment (start 227.965 54.2925) (end 227.965 47.02) (width 1) (layer "F.Cu") (net 2))
   (segment (start 222.25 60.0075) (end 227.965 54.2925) (width 1) (layer "F.Cu") (net 2))
@@
   (segment (start 197.485 38.735) (end 200.66 35.56) (width 1) (layer "F.Cu") (net 9))
   (segment (start 205.73 63.49) (end 197.485 55.245) (width 1) (layer "F.Cu") (net 9))
-  (segment (start 208.28 38.1) (end 213.36 38.1) (width 1) (layer "F.Cu") (net 10))
-  (segment (start 231.215 32.675) (end 224.715 32.675) (width 1) (layer "F.Cu") (net 10))
   (segment (start 207.645 60.95) (end 205.73 60.95) (width 1) (layer "F.Cu") (net 10))
   (segment (start 201.295 38.1) (end 201.93 38.1) (width 1) (layer "F.Cu") (net 10))
+  (segment (start 231.215 37.175) (end 224.715 37.175) (width 1) (layer "F.Cu") (net 10))
+  (segment (start 220 37.175) (end 224.715 37.175) (width 1) (layer "F.Cu") (net 10))
+  (segment (start 208.28 38.1) (end 219.075 38.1) (width 1) (layer "F.Cu") (net 10))
   (segment (start 199.39 54.61) (end 199.39 40.005) (width 1) (layer "F.Cu") (net 10))
   (segment (start 208.28 38.1) (end 201.93 38.1) (width 1) (layer "F.Cu") (net 10))
   (segment (start 199.39 40.005) (end 201.295 38.1) (width 1) (layer "F.Cu") (net 10))
-  (segment (start 218.785 32.675) (end 224.715 32.675) (width 1) (layer "F.Cu") (net 10))
-  (segment (start 213.36 38.1) (end 218.785 32.675) (width 1) (layer "F.Cu") (net 10))
+  (segment (start 219.075 38.1) (end 220 37.175) (width 1) (layer "F.Cu") (net 10))
   (segment (start 205.73 60.95) (end 199.39 54.61) (width 1) (layer "F.Cu") (net 10))
-  (segment (start 218.7575 62.5475) (end 217.17 64.135) (width 1) (layer "F.Cu") (net 12))
-  (segment (start 209.803299 64.77) (end 211.455 64.77) (width 0.25) (layer "F.Cu") (net 12))
-  (segment (start 209.01 63.976701) (end 209.803299 64.77) (width 0.25) (layer "F.Cu") (net 12))
-  (segment (start 222.25 62.5475) (end 218.7575 62.5475) (width 1) (layer "F.Cu") (net 12))
-  (segment (start 207.645 58.41) (end 209.01 59.775) (width 0.25) (layer "F.Cu") (net 12))
-  (segment (start 217.17 64.135) (end 212.09 64.135) (width 1) (layer "F.Cu") (net 12))
-  (segment (start 209.01 59.775) (end 209.01 63.976701) (width 0.25) (layer "F.Cu") (net 12))
+  (segment (start 213.6775 62.5475) (end 212.09 60.96) (width 1) (layer "F.Cu") (net 12))
   (segment (start 207.645 58.41) (end 208.2725 58.41) (width 0.25) (layer "F.Cu") (net 12))
-  (segment (start 211.455 64.77) (end 212.09 64.135) (width 0.25) (layer "F.Cu") (net 12))
+  (segment (start 207.645 58.41) (end 208.82 59.585) (width 0.25) (layer "F.Cu") (net 12))
+  (segment (start 210.715 59.585) (end 212.09 60.96) (width 0.25) (layer "F.Cu") (net 12))
+  (segment (start 208.82 59.585) (end 210.715 59.585) (width 0.25) (layer "F.Cu") (net 12))
+  (segment (start 222.25 62.5475) (end 213.6775 62.5475) (width 1) (layer "F.Cu") (net 12))
   (zone (net 1) (net_name "+3.3V") (layer "F.Cu") (hatch edge 0.5)
     (priority 1)

Commit message: minor change to fit OLED screen connector
Parts:
- J5: value Aux_I2C -> Display
- moved C3 6.25 mm to (205.7, 41.9)
Connections:
- J5 pad 1: +3.3V -> GND
- J5 pad 2: GND -> +3.3V
Routing:
- net +3.3V: track 55.6 -> 66.6 mm
- net GND: track 30.0 -> 29.7 mm, vias 16 -> 14
Other:
- outline, holes or cut-outs redrawn
- board text added: "3.3V"
- board text added: "GND"
- board text added: "SCL"
- board text added: "SDA"
- board text added: "WiFi Temp Sensor V0_3 Rich Clubb https://github.com/richClubb/wifi_temp_sensor"
Changed lines of the file:
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@@
     (property "ki_keywords" "connector")
     (attr through_hole)
-    (fp_text reference "J5" (at -2.54 -1.27) (layer "F.SilkS")
-        (effects (font (size 1 1) (thickness 0.15)))
-    )
-    (fp_text value "Aux_I2C" (at 0 10.39) (layer "F.Fab")
+    (fp_text reference "J5" (at -2.54 -1.905) (layer "F.SilkS")
+        (effects (font (size 1 1) (thickness 0.15)))
+    )
+    (fp_text value "Display" (at 0 10.39) (layer "F.Fab")
         (effects (font (size 1 1) (thickness 0.15)))
     )
@@
       (stroke (width 0.1) (type solid)) (layer "F.Fab"))
     (pad "1" thru_hole rect (at 0 0 180) (size 1.7 1.7) (drill 1) (layers "*.Cu" "*.Mask")
-      (net 1 "+3.3V") (pinfunction "Pin_1") (pintype "passive"))
+      (net 6 "GND") (pinfunction "Pin_1") (pintype "passive"))
     (pad "2" thru_hole oval (at 0 2.54 180) (size 1.7 1.7) (drill 1) (layers "*.Cu" "*.Mask")
-      (net 6 "GND") (pinfunction "Pin_2") (pintype "passive"))
+      (net 1 "+3.3V") (pinfunction "Pin_2") (pintype "passive"))
     (pad "3" thru_hole oval (at 0 5.08 180) (size 1.7 1.7) (drill 1) (layers "*.Cu" "*.Mask")
       (net 10 "SCL") (pinfunction "Pin_3") (pintype "passive"))
@@
   )
   (footprint "Capacitor_SMD:C_1206_3216Metric" (layer "F.Cu")
-    (at 208.28 47.625 -90)
+    (at 205.74 41.91 -90)
     (descr "Capacitor SMD 1206 (3216 Metric), square (rectangular) end terminal, IPC_7351 nominal, (Body size source: IPC-SM-782 page 76, https://www.pcb-3d.com/wordpress/wp-content/uploads/ipc-sm-782a_amendment_1_and_2.pdf), generated with kicad-footprint-generator")
     (tags "capacitor")
@@
     (property "ki_keywords" "connector")
     (attr through_hole)
-    (fp_text reference "J3" (at 2.54 0) (layer "F.SilkS")
+    (fp_text reference "J3" (at -2.54 -1.905) (layer "F.SilkS")
         (effects (font (size 1 1) (thickness 0.15)))
     )
@@
     )
   )
+  (gr_circle (center 230.505 28.575) (end 233.045 28.575)
+    (stroke (width 0.2) (type default)) (fill none) (layer "B.Cu"))
+  (gr_circle (center 230.505 66.675) (end 233.045 66.675)
+    (stroke (width 0.1) (type default)) (fill none) (layer "B.Cu"))
+  (gr_circle (center 187.32942 66.675) (end 189.87384 66.675)
+    (stroke (width 0.1) (type default)) (fill none) (layer "B.Cu"))
+  (gr_circle (center 187.325 28.575) (end 189.865 28.575)
+    (stroke (width 0.2) (type default)) (fill none) (layer "B.Cu"))
   (gr_rect (start 189.23 27.305) (end 205.105 52.705)
     (stroke (width 0.2) (type default)) (fill none) (layer "F.SilkS"))
@@
   (gr_circle (center 230.505 66.675) (end 231.924903 66.675)
     (stroke (width 0.2) (type default)) (fill none) (layer "Edge.Cuts"))
+  (gr_circle (center 187.325 66.675) (end 186.69 65.405)
+    (stroke (width 0.1) (type default)) (fill none) (layer "Edge.Cuts"))
   (gr_line (start 183.515 70.485) (end 234.315 70.485)
     (stroke (width 0.1) (type default)) (layer "Edge.Cuts"))
@@
   (gr_line (start 234.315 24.765) (end 183.515 24.765)
     (stroke (width 0.1) (type default)) (layer "Edge.Cuts"))
-  (gr_circle (center 187.175097 66.675) (end 188.595 66.675)
-    (stroke (width 0.2) (type default)) (fill none) (layer "Edge.Cuts"))
   (gr_line (start 183.515 24.765) (end 183.515 70.485)
     (stroke (width 0.1) (type default)) (layer "Edge.Cuts"))
+  (gr_text "WiFi Temp Sensor V0_3\nRich Clubb\nhttps://github.com/richClubb/wifi_temp_sensor" (at 227.33 31.115) (layer "B.SilkS")
+    (effects (font (size 1 1) (thickness 0.15)) (justify left bottom mirror))
+  )
+  (gr_text "SDA" (at 209.55 36.195) (layer "F.SilkS")
+    (effects (font (size 1 1) (thickness 0.25) bold) (justify left bottom))
+  )
+  (gr_text "SDA" (at 202.565 64.135) (layer "F.SilkS")
+    (effects (font (size 1 1) (thickness 0.25) bold) (justify left bottom))
+  )
+  (gr_text "SCL" (at 197.485 38.735) (layer "F.SilkS")
+    (effects (font (size 1 1) (thickness 0.25) bold) (justify left bottom))
+  )
+  (gr_text "GND" (at 196.85 41.275) (layer "F.SilkS")
+    (effects (font (size 1 1) (thickness 0.25) bold) (justify left bottom))
+  )
+  (gr_text "SCL" (at 202.565 61.595) (layer "F.SilkS")
+    (effects (font (size 1 1) (thickness 0.25) bold) (justify left bottom))
+  )
+  (gr_text "3.3V" (at 196.85 43.815) (layer "F.SilkS")
+    (effects (font (size 1 1) (thickness 0.25) bold) (justify left bottom))
+  )
+  (gr_text "GND" (at 209.55 43.815) (layer "F.SilkS")
+    (effects (font (size 1 1) (thickness 0.25) bold) (justify left bottom))
+  )
+  (gr_text "SCL" (at 209.55 38.735) (layer "F.SilkS")
+    (effects (font (size 1 1) (thickness 0.25) bold) (justify left bottom))
+  )
+  (gr_text "SDA" (at 197.485 36.195) (layer "F.SilkS")
+    (effects (font (size 1 1) (thickness 0.25) bold) (justify left bottom))
+  )
+  (gr_text "3.3V" (at 209.55 41.275) (layer "F.SilkS")
+    (effects (font (size 1 1) (thickness 0.25) bold) (justify left bottom))
+  )
   (segment (start 201.93 43.18) (end 201.93 46.15) (width 1) (layer "F.Cu") (net 1))
   (segment (start 210.195 63.5) (end 210.185 63.49) (width 0.5) (layer "F.Cu") (net 1))
@@
   (segment (start 213.995 58.625) (end 216.535 56.085) (width 1) (layer "F.Cu") (net 1))
   (segment (start 216.535 46.67) (end 217.485 45.72) (width 1) (layer "F.Cu") (net 1))
-  (segment (start 217.485 45.72) (end 218.3975 45.72) (width 1) (layer "F.Cu") (net 1))
   (segment (start 201.93 46.15) (end 208.28 46.15) (width 1) (layer "F.Cu") (net 1))
-  (segment (start 208.28 43.18) (end 208.28 46.15) (width 1) (layer "F.Cu") (net 1))
   (segment (start 213.78 58.41) (end 213.995 58.625) (width 1) (layer "F.Cu") (net 1))
   (segment (start 220.345 45.72) (end 218.3975 45.72) (width 0.5) (layer "F.Cu") (net 1))
+  (segment (start 205.74 40.435) (end 208.075 40.435) (width 1) (layer "F.Cu") (net 1))
   (segment (start 212.715 63.49) (end 212.725 63.5) (width 0.25) (layer "F.Cu") (net 1))
   (segment (start 215.9 45.72) (end 218.3975 45.72) (width 0.5) (layer "F.Cu") (net 1))
+  (segment (start 212.405 40.64) (end 217.485 45.72) (width 1) (layer "F.Cu") (net 1))
   (segment (start 208.71 45.72) (end 218.3975 45.72) (width 1) (layer "F.Cu") (net 1))
+  (segment (start 208.075 40.435) (end 208.28 40.64) (width 1) (layer "F.Cu") (net 1))
   (segment (start 212.725 63.5) (end 210.195 63.5) (width 0.5) (layer "F.Cu") (net 1))
+  (segment (start 217.485 45.72) (end 218.3975 45.72) (width 1) (layer "F.Cu") (net 1))
   (segment (start 221.66 46.125) (end 220.75 46.125) (width 0.5) (layer "F.Cu") (net 1))
   (segment (start 208.28 46.15) (end 208.71 45.72) (width 1) (layer "F.Cu") (net 1))
+  (segment (start 208.28 40.64) (end 212.405 40.64) (width 1) (layer "F.Cu") (net 1))
   (segment (start 220.75 46.125) (end 220.345 45.72) (width 0.5) (layer "F.Cu") (net 1))
   (via (at 213.995 60.325) (size 0.8) (drill 0.4) (layers "F.Cu" "B.Cu") (free) (net 1))
@@
   (segment (start 201.93 50.165) (end 201.295 50.8) (width 1) (layer "F.Cu") (net 6))
   (segment (start 218.485 47.22) (end 218.485 48.305) (width 1) (layer "F.Cu") (net 6))
-  (segment (start 208.28 49.1) (end 208.28 50.165) (width 1) (layer "F.Cu") (net 6))
   (segment (start 226.06 44.45) (end 226.06 43.18) (width 0.5) (layer "F.Cu") (net 6))
   (segment (start 201.93 50.165) (end 202.565 50.8) (width 1) (layer "F.Cu") (net 6))
@@
   (segment (start 201.93 49.1) (end 201.93 50.165) (width 1) (layer "F.Cu") (net 6))
   (segment (start 226.06 44.45) (end 227.33 44.45) (width 0.5) (layer "F.Cu") (net 6))
-  (segment (start 208.28 50.165) (end 208.915 50.8) (width 1) (layer "F.Cu") (net 6))
-  (segment (start 208.28 50.165) (end 207.645 50.8) (width 1) (layer "F.Cu") (net 6))
   (segment (start 221.66 41.27) (end 221.66 39.96) (width 1) (layer "F.Cu") (net 6))
+  (segment (start 208.28 43.18) (end 205.945 43.18) (width 1) (layer "F.Cu") (net 6))
   (segment (start 228.6 44.42) (end 228.57 44.42) (width 0.5) (layer "F.Cu") (net 6))
   (segment (start 218.485 48.215) (end 217.805 48.895) (width 1) (layer "F.Cu") (net 6))
   (segment (start 218.485 47.22) (end 218.485 48.215) (width 1) (layer "F.Cu") (net 6))
   (segment (start 221.66 49.075) (end 221.66 50.12) (width 1) (layer "F.Cu") (net 6))
+  (segment (start 205.945 43.18) (end 205.74 43.385) (width 1) (layer "F.Cu") (net 6))
   (segment (start 221.66 41.27) (end 221.66 40.05) (width 1) (layer "F.Cu") (net 6))
   (segment (start 221.66 40.05) (end 220.98 39.37) (width 1) (layer "F.Cu") (net 6))
@@
   (via (at 226.06 44.45) (size 0.8) (drill 0.4) (layers "F.Cu" "B.Cu") (free) (net 6))
   (via (at 220.98 50.8) (size 0.8) (drill 0.4) (layers "F.Cu" "B.Cu") (free) (net 6))
-  (via (at 207.645 50.8) (size 0.8) (drill 0.4) (layers "F.Cu" "B.Cu") (free) (net 6))
   (via (at 227.33 44.45) (size 0.8) (drill 0.4) (layers "F.Cu" "B.Cu") (free) (net 6))
   (via (at 227.33 43.18) (size 0.8) (drill 0.4) (layers "F.Cu" "B.Cu") (free) (net 6))
   (via (at 201.295 50.8) (size 0.8) (drill 0.4) (layers "F.Cu" "B.Cu") (free) (net 6))
   (via (at 217.805 48.895) (size 0.8) (drill 0.4) (layers "F.Cu" "B.Cu") (free) (net 6))
-  (via (at 208.915 50.8) (size 0.8) (drill 0.4) (layers "F.Cu" "B.Cu") (free) (net 6))
   (via (at 226.06 43.18) (size 0.8) (drill 0.4) (layers "F.Cu" "B.Cu") (free) (net 6))
   (via (at 222.25 39.37) (size 0.8) (drill 0.4) (layers "F.Cu" "B.Cu") (free) (net 6))
